File: PCB Mestrado/STLINK.kicad_sch (KiCad schematic)
At the start: 32 parts, among them P1 USB_C_Plug, Q1 BC817, U1 STM32F103CBTx, Y2 8MHz

Commit message: BUILDING
Parts:
- removed C25: 100nF, Capacitor_SMD:C_0603_1608Metric, symbol Device:C
Changed lines of the file:
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@@
   (junction (at 36.83 50.8) (diameter 0) (color 0 0 0 0)
   )
-  (junction (at 148.59 30.48) (diameter 0) (color 0 0 0 0)
-  )
   (junction (at 78.74 93.98) (diameter 0) (color 0 0 0 0)
   )
@@
   (junction (at 279.4 144.78) (diameter 0) (color 0 0 0 0)
   )
-  (junction (at 148.59 22.86) (diameter 0) (color 0 0 0 0)
-  )
   (junction (at 59.69 50.8) (diameter 0) (color 0 0 0 0)
   )
@@
     (stroke (width 0) (type default) (color 0 0 0 0))
   )
-  (wire (pts (xy 148.59 30.48) (xy 160.02 30.48))
-    (stroke (width 0) (type default) (color 0 0 0 0))
-  )
   (wire (pts (xy 106.68 99.06) (xy 105.41 99.06))
     (stroke (width 0) (type default) (color 0 0 0 0))
@@
   )
   (wire (pts (xy 176.53 101.6) (xy 179.07 101.6))
-    (stroke (width 0) (type default) (color 0 0 0 0))
-  )
-  (wire (pts (xy 148.59 22.86) (xy 160.02 22.86))
     (stroke (width 0) (type default) (color 0 0 0 0))
   )
@@
       (effects (font (size 1.27 1.27)) hide)
     )
-    (pin "1")
-    (pin "2")
-  )
-  (symbol (lib_id "Device:C") (at 160.02 26.67 0) (unit 1)
-    (in_bom yes) (on_board yes) (fields_autoplaced)
-    (property "Reference" "C25" (id 0) (at 163.83 25.3999 0)
-      (effects (font (size 1.27 1.27)) (justify left))
-    )
-    (property "Value" "100nF" (id 1) (at 163.83 27.9399 0)
-      (effects (font (size 1.27 1.27)) (justify left))
-    )
-    (property "Footprint" "Capacitor_SMD:C_0603_1608Metric" (id 2) (at 160.9852 30.48 0)
-      (effects (font (size 1.27 1.27)) hide)
-    )
-    (property "Datasheet" "~" (id 3) (at 160.02 26.67 0)
-      (effects (font (size 1.27 1.27)) hide)
-    )
-    (property "LCSC Part" "C14663" (id 4) (at 160.02 26.67 0)
-      (effects (font (size 1.27 1.27)) hide)
-    )
