File: PCB Mestrado/MOTOR.kicad_sch (KiCad schematic)
At the start: 19 parts, among them J1 Conn_01x02_Female, U3 MC33926, U7 MCR1101-XX-3

Commit message: BUILDING
Parts:
- added J3: Jack-DC, Connector_BarrelJack:BarrelJack_GCT_DCJ200-10-A_Horizontal, symbol Connector:Jack-DC
- C26, C28: footprint Capacitor_SMD:C_1206_3216Metric -> Capacitor_SMD:C_0603_1608Metric
Connections:
- net 12V: now also J3.1
- net GNDD: now also J3.2
- net M1: now also J1.2 (Pin_2); no longer J1.1 (Pin_1)
- net M2: now also J1.1 (Pin_1); no longer J1.2 (Pin_2)
- net MID_M: now reaches U3.12 (OUT1), U3.13 (OUT1), U3.14 (OUT1), U3.15 (OUT1), U7.1 (IP+), U7.2 (IP+), U7.3 (IP+), U7.4 (IP+)
Other:
- moved on the sheet: J1
Changed lines of the file:
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@@
+    (stroke (width 0) (type default) (color 0 0 0 0))
+  )
+  (wire (pts (xy 199.39 90.17) (xy 168.91 90.17))
     (stroke (width 0) (type default) (color 0 0 0 0))
   )
@@
     (stroke (width 0) (type default) (color 0 0 0 0))
   )
-  (wire (pts (xy 168.91 88.9) (xy 199.39 88.9))
-    (stroke (width 0) (type default) (color 0 0 0 0))
-  )
   (wire (pts (xy 102.87 64.77) (xy 107.95 64.77))
     (stroke (width 0) (type default) (color 0 0 0 0))
@@
     (stroke (width 0) (type default) (color 0 0 0 0))
   )
+  (wire (pts (xy 33.02 123.19) (xy 43.18 123.19))
+    (stroke (width 0) (type default) (color 0 0 0 0))
+  )
   (wire (pts (xy 102.87 31.75) (xy 105.41 31.75))
     (stroke (width 0) (type default) (color 0 0 0 0))
@@
     (stroke (width 0) (type default) (color 0 0 0 0))
   )
-  (wire (pts (xy 199.39 86.36) (xy 194.31 86.36))
-    (stroke (width 0) (type default) (color 0 0 0 0))
-  )
-  (wire (pts (xy 168.91 81.28) (xy 168.91 88.9))
+  (wire (pts (xy 168.91 81.28) (xy 168.91 90.17))
     (stroke (width 0) (type default) (color 0 0 0 0))
   )
@@
     (stroke (width 0) (type default) (color 0 0 0 0))
   )
+  (wire (pts (xy 33.02 120.65) (xy 39.37 120.65))
+    (stroke (width 0) (type default) (color 0 0 0 0))
+  )
   (wire (pts (xy 204.47 54.61) (xy 200.66 54.61))
     (stroke (width 0) (type default) (color 0 0 0 0))
@@
     (stroke (width 0) (type default) (color 0 0 0 0))
   )
+  (wire (pts (xy 43.18 123.19) (xy 43.18 125.73))
+    (stroke (width 0) (type default) (color 0 0 0 0))
+  )
   (wire (pts (xy 80.01 72.39) (xy 82.55 72.39))
     (stroke (width 0) (type default) (color 0 0 0 0))
   )
+  (wire (pts (xy 194.31 87.63) (xy 199.39 87.63))
+    (stroke (width 0) (type default) (color 0 0 0 0))
+  )
   (wire (pts (xy 58.42 69.85) (xy 58.42 68.58))
     (stroke (width 0) (type default) (color 0 0 0 0))
@@
     (stroke (width 0) (type default) (color 0 0 0 0))
   )
+  (wire (pts (xy 39.37 116.84) (xy 40.64 116.84))
+    (stroke (width 0) (type default) (color 0 0 0 0))
+  )
   (wire (pts (xy 80.01 74.93) (xy 80.01 77.47))
     (stroke (width 0) (type default) (color 0 0 0 0))
@@
     (stroke (width 0) (type default) (color 0 0 0 0))
   )
+  (wire (pts (xy 39.37 120.65) (xy 39.37 116.84))
+    (stroke (width 0) (type default) (color 0 0 0 0))
+  )
   (wire (pts (xy 107.95 71.12) (xy 107.95 68.58))
     (stroke (width 0) (type default) (color 0 0 0 0))
   )
-  (wire (pts (xy 194.31 86.36) (xy 194.31 77.47))
+  (wire (pts (xy 194.31 77.47) (xy 194.31 87.63))
     (stroke (width 0) (type default) (color 0 0 0 0))
   )
@@
   )
   (wire (pts (xy 200.66 50.8) (xy 200.66 48.26))
+    (stroke (width 0) (type default) (color 0 0 0 0))
+  )
+  (wire (pts (xy 33.02 123.19) (xy 33.02 125.73))
     (stroke (width 0) (type default) (color 0 0 0 0))
   )
@@
     )
   )
+  (global_label "12V" (shape input) (at 40.64 116.84 0) (fields_autoplaced)
+    (effects (font (size 1.27 1.27)) (justify left))
+    (property "Intersheet References" "${INTERSHEET_REFS}" (id 0) (at 46.5607 116.9194 0)
+      (effects (font (size 1.27 1.27)) (justify left) hide)
+    )
+  )
   (global_label "VCC" (shape input) (at 78.74 21.59 90) (fields_autoplaced)
     (effects (font (size 1.27 1.27)) (justify left))
@@
     )
   )
+  (global_label "MID_M" (shape input) (at 168.91 43.18 90) (fields_autoplaced)
+    (effects (font (size 1.27 1.27)) (justify left))
+    (property "Intersheet References" "${INTERSHEET_REFS}" (id 0) (at 168.8306 35.0217 90)
+      (effects (font (size 1.27 1.27)) (justify left) hide)
+    )
+  )
   (global_label "D2" (shape input) (at 60.96 41.91 180) (fields_autoplaced)
     (effects (font (size 1.27 1.27)) (justify right))
@@
       (effects (font (size 1.27 1.27)) (justify left))
     )
-    (property "Footprint" "Capacitor_SMD:C_1206_3216Metric" (id 2) (at 59.3852 68.58 0)
+    (property "Footprint" "Capacitor_SMD:C_0603_1608Metric" (id 2) (at 59.3852 68.58 0)
       (effects (font (size 1.27 1.27)) hide)
     )
@@
     (pin "1")
   )
-  (symbol (lib_id "Connector:Conn_01x02_Female") (at 204.47 86.36 0) (unit 1)
-    (in_bom yes) (on_board yes) (fields_autoplaced)
-    (property "Reference" "J1" (id 0) (at 205.74 86.3599 0)
-      (effects (font (size 1.27 1.27)) (justify left))
-    )
-    (property "Value" "Conn_01x02_Female" (id 1) (at 205.74 88.8999 0)
-      (effects (font (size 1.27 1.27)) (justify left))
-    )
-    (property "Footprint" "Connector_Phoenix_MSTB:PhoenixContact_MSTBA_2,5_2-G-5,08_1x02_P5.08mm_Horizontal" (id 2) (at 204.47 86.36 0)
-      (effects (font (size 1.27 1.27)) hide)
-    )
-    (property "Datasheet" "~" (id 3) (at 204.47 86.36 0)
+  (symbol (lib_id "Connector:Conn_01x02_Female") (at 204.47 90.17 0) (mirror x) (unit 1)
+    (in_bom yes) (on_board yes) (fields_autoplaced)
+    (property "Reference" "J1" (id 0) (at 203.835 82.55 0))
+    (property "Value" "Conn_01x02_Female" (id 1) (at 203.835 85.09 0))
+    (property "Footprint" "Connector_Phoenix_MSTB:PhoenixContact_MSTBA_2,5_2-G-5,08_1x02_P5.08mm_Horizontal" (id 2) (at 204.47 90.17 0)
+      (effects (font (size 1.27 1.27)) hide)
+    )
+    (property "Datasheet" "~" (id 3) (at 204.47 90.17 0)
       (effects (font (size 1.27 1.27)) hide)
     )
@@
     (property "Reference" "C28" (id 0) (at 247.65 43.18 90))
     (property "Value" "10nF" (id 1) (at 247.65 45.72 90))
-    (property "Footprint" "Capacitor_SMD:C_1206_3216Metric" (id 2) (at 251.46 49.8348 0)
+    (property "Footprint" "Capacitor_SMD:C_0603_1608Metric" (id 2) (at 251.46 49.8348 0)
       (effects (font (size 1.27 1.27)) hide)
     )
@@
     (pin "2")
   )
+  (symbol (lib_id "Connector:Jack-DC") (at 25.4 123.19 0) (unit 1)
+    (in_bom yes) (on_board yes) (fields_autoplaced)
+    (property "Reference" "J3" (id 0) (at 25.4 114.3 0))
+    (property "Value" "Jack-DC" (id 1) (at 25.4 116.84 0))
+    (property "Footprint" "Connector_BarrelJack:BarrelJack_GCT_DCJ200-10-A_Horizontal" (id 2) (at 26.67 124.206 0)
+      (effects (font (size 1.27 1.27)) hide)
+    )
+    (property "Datasheet" "~" (id 3) (at 26.67 124.206 0)
+      (effects (font (size 1.27 1.27)) hide)
+    )
+    (pin "1")
+    (pin "2")
+  )
   (symbol (lib_id "Device:R") (at 250.19 38.1 270) (mirror x) (unit 1)
     (in_bom yes) (on_board yes) (fields_autoplaced)
@@
     (pin "2")
   )
+  (symbol (lib_id "power:GNDD") (at 43.18 125.73 0) (unit 1)
+    (in_bom yes) (on_board yes) (fields_autoplaced)
+    (property "Reference" "#PWR0131" (id 0) (at 43.18 132.08 0)
+      (effects (font (size 1.27 1.27)) hide)
+    )
+    (property "Value" "GNDD" (id 1) (at 43.18 130.81 0))
+    (property "Footprint" "" (id 2) (at 43.18 125.73 0)
+      (effects (font (size 1.27 1.27)) hide)
+    )
+    (property "Datasheet" "" (id 3) (at 43.18 125.73 0)
+      (effects (font (size 1.27 1.27)) hide)
+    )
+    (pin "1")
+  )
   (symbol (lib_id "Device:R") (at 67.31 38.1 270) (mirror x) (unit 1)

Commit message: build
Connections:
- net VCC renamed VDD
Changed lines of the file:
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@@
     )
   )
-  (global_label "VCC" (shape input) (at 78.74 21.59 90) (fields_autoplaced)
+  (global_label "VDD" (shape input) (at 78.74 21.59 90) (fields_autoplaced)
     (effects (font (size 1.27 1.27)) (justify left))
     (property "Intersheet References" "${INTERSHEET_REFS}" (id 0) (at 78.6606 15.5483 90)
@@
     )
   )
-  (global_label "VCC" (shape input) (at 254 60.96 0) (fields_autoplaced)
+  (global_label "VDD" (shape input) (at 254 60.96 0) (fields_autoplaced)
     (effects (font (size 1.27 1.27)) (justify left))
     (property "Intersheet References" "${INTERSHEET_REFS}" (id 0) (at 260.0417 60.8806 0)
@@
     )
   )
-  (global_label "VCC" (shape input) (at 256.54 38.1 0) (fields_autoplaced)
+  (global_label "VDD" (shape input) (at 256.54 38.1 0) (fields_autoplaced)
     (effects (font (size 1.27 1.27)) (justify left))
     (property "Intersheet References" "${INTERSHEET_REFS}" (id 0) (at 262.5817 38.0206 0)
@@
     )
   )
-  (global_label "VCC" (shape input) (at 226.06 58.42 0) (fields_autoplaced)
+  (global_label "VDD" (shape input) (at 226.06 58.42 0) (fields_autoplaced)
     (effects (font (size 1.27 1.27)) (justify left))
     (property "Intersheet References" "${INTERSHEET_REFS}" (id 0) (at 232.1017 58.3406 0)
