File: PCB Mestrado/PCBMestrado_v1.kicad_pcb (KiCad board)
At the start: 2 copper layers, 100 x 100 mm, 102 parts, among them J1 Conn_01x02_Female, J2 USB_C_Receptacle_USB2.0, P1 USB_C_Plug, Q1 BC817, SW1 SW_Push_Dual, SW2 SW_Push_Dual, U1 STM32F103CBTx, U2 STM32F446RETx, U3 MC33926, U4 AMS1117-3.3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

Commit message: BUILDING
Parts:
- removed C12, C25: 100nF, Capacitor_SMD:C_0603_1608Metric
- removed D4: MBR0540, Diode_SMD:D_SOD-123
- removed R22: 8K2, Resistor_SMD:R_0603_1608Metric
- removed R4: 47K, Resistor_SMD:R_0603_1608Metric
- added J3: Jack-DC, Connector_BarrelJack:BarrelJack_GCT_DCJ200-10-A_Horizontal, F.Cu at (114.1, 80.2)
- added J4: Conn_01x02_Female, Connector_Phoenix_MSTB:PhoenixContact_MSTBA_2,5_2-G-5,08_1x02_P5.08mm_Horizontal, F.Cu at (110.2, 92.3)
- added J5: Conn_01x04_Male, Connector_JST:JST_EH_B4B-EH-A_1x04_P2.50mm_Vertical, F.Cu at (135.8, 148.5)
- added J6: Conn_01x04_Male, Connector_JST:JST_EH_B4B-EH-A_1x04_P2.50mm_Vertical, F.Cu at (121.5, 148.5)
- added JP1: Jumper_3_Open, Jumper:SolderJumper-3_P2.0mm_Open_TrianglePad1.0x1.5mm, F.Cu at (141.1, 147.4)
- added JP2: Jumper_3_Open, Jumper:SolderJumper-3_P2.0mm_Open_TrianglePad1.0x1.5mm, F.Cu at (119.9, 144.1)
- C26, C28: footprint Capacitor_SMD:C_1206_3216Metric -> Capacitor_SMD:C_0603_1608Metric
- moved R16 117.9 mm to (116.2, 94.5), turned to -90 degrees
- moved C9 109.4 mm to (128.0, 94.8), turned to -90 degrees
- moved U6 108.7 mm to (122.7, 94.7), turned to 180 degrees
- moved R19 86.5 mm to (153.6, 83.7)
- moved R3 85.1 mm to (159.1, 66.1)
- moved R8 84.6 mm to (157.2, 148.5), turned to 180 degrees
- moved R2 84.2 mm to (159.1, 64.5)
- moved D5 84.0 mm to (153.9, 148.5), turned to 180 degrees
- moved SW2 80.1 mm to (147.4, 83.5), turned to 180 degrees
- moved R7 79.1 mm to (157.3, 146.8), turned to 180 degrees
- moved R5 78.1 mm to (167.3, 62.2)
- moved R1 77.4 mm to (153.6, 85.4), turned to 180 degrees
- moved R6 74.3 mm to (167.3, 63.8)
- moved D3 68.9 mm to (153.9, 146.8), turned to 180 degrees
- moved D1 68.7 mm to (172.7, 64.4)
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Connections:
- net Net-(U3-Pad12) renamed MID_M
- J1 pad 1: M1 -> M2
- J1 pad 2: M2 -> M1
Routing:
- net VDD: track 212.8 -> 624.7 mm, vias 6 -> 14
- net 5V: track 44.6 -> 300.2 mm, vias 1 -> 12
- net 12V: track 7.64 -> 172.7 mm, vias 0 -> 11
- net SF: track 13.7 -> 89.7 mm, vias 0 -> 4
- net STLINK_TX: track 20.9 -> 96.2 mm, vias 0 -> 1
- net D1: track 13.8 -> 75.5 mm, vias 0 -> 2
- net D2: track 21.4 -> 81.6 mm, vias 0 -> 4
- net USB_D+: track 17.0 -> 76.0 mm
- net USB_D-: track 16.2 -> 75.1 mm
- net STLINK_USB_D+: track 0.00 -> 55.3 mm, vias 0 -> 3
- net STLINK_RENUN: track 0.00 -> 54.6 mm, vias 0 -> 2
- net FB_DRIVER: track 18.0 -> 71.4 mm, vias 0 -> 2
- net Net-(R3-Pad2): track 17.9 -> 68.1 mm, vias 0 -> 1
- net INV: track 19.7 -> 69.9 mm, vias 0 -> 2
- net EN: track 18.2 -> 67.0 mm, vias 0 -> 3
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- added copper zone on B.Cu, net GNDD
- added copper zone on F.Cu, net GNDD
- added copper zone on F.Cu, net M1
- added copper zone on F.Cu, net M2
- added copper zone on F.Cu, net MID_M

Commit message: build
Parts:
- removed D5: LED, LED_SMD:LED_0603_1608Metric
- removed R8: 680R, Resistor_SMD:R_0603_1608Metric
- added D4: LED, LED_SMD:LED_0603_1608Metric, F.Cu at (167.9, 145.5)
- added J7: Conn_01x08_Female, Connector_JST:JST_EH_B8B-EH-A_1x08_P2.50mm_Vertical, F.Cu at (190.1, 117.9)
- added R4: 680R, Resistor_SMD:R_0603_1608Metric, F.Cu at (171.4, 148.1)
- moved R7 14.2 mm to (171.4, 145.5)
- moved D3 14.0 mm to (167.9, 148.1)
- moved R5 2.45 mm to (167.6, 64.7), turned to 90 degrees
- moved R6 2.14 mm to (169.3, 64.7), turned to 90 degrees
- moved JP2 1.71 mm to (121.6, 144.2)
- moved J2 0.23 mm to (172.0, 55.2)
Connections:
- D3 pad 2: Net-(D3-Pad2) -> Net-(U2-Pad24)
- R46 pad 1: VCC -> VDD
- R48 pad 1: VCC -> VDD
- R49 pad 1: VCC -> VDD
- R7 pad 2: Net-(D3-Pad1) -> Net-(D4-Pad1)
- U2 pad 17: unconnected-(U2-Pad17) -> STLINK_RX
- U2 pad 20: Net-(D5-Pad2) -> unconnected-(U2-Pad20)
- U2 pad 21: Net-(D3-Pad2) -> unconnected-(U2-Pad21)
- U2 pad 24: unconnected-(U2-Pad24) -> Net-(U2-Pad24)
- U2 pad 25: unconnected-(U2-Pad25) -> Net-(U2-Pad25)
- U7 pad 10: VCC -> VDD
Routing:
- net STLINK_RX: track 0.00 -> 104.7 mm, vias 0 -> 2
- net VDD: track 624.7 -> 721.6 mm, vias 14 -> 19
- net VCC: track 45.1 -> 0.00 mm, vias 4 -> 0
- net Net-(D5-Pad2): track 28.4 -> 0.00 mm
- net Net-(U2-Pad24): track 0.00 -> 27.3 mm
- net Net-(D3-Pad2): track 24.1 -> 0.00 mm
- net DC_LCD: track 21.0 -> 44.9 mm, vias 0 -> 2
- net Net-(U2-Pad25): track 0.00 -> 23.0 mm
- net unconnected-(U2-Pad17): track 23.0 -> 0.00 mm
- net unconnected-(U2-Pad20): track 0.00 -> 20.5 mm
- net unconnected-(U2-Pad21): track 0.00 -> 19.6 mm
- net unconnected-(U2-Pad24): track 17.1 -> 0.00 mm
- net unconnected-(U2-Pad25): track 16.9 -> 0.00 mm
- net CS_LCD_1: track 16.4 -> 32.6 mm
- net SCK_LCD: track 20.3 -> 31.9 mm
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Other:
- outline, holes or cut-outs redrawn
- board text added: "CAN BUS"
- board text added: "ENCODER"
- board text added: "LCD"
- board text added: "LED1"
- board text added: "LED2"
- board text added: "MOTOR DRIVER"
- board text added: "POWER SUPPLY"
- board text added: "STLINK"
- board text added: "TPS"
- board text added: "VIN"
